Commit message: Leds NOT WORKING ALONE. Only with cameragit add ../build/monkey

File: swarm_clover_description/urdf/clover/clover4.xacro (robot description, xacro)
@@ -38,6 +38,6 @@
         <name>gps0</name>
       </include>
-      <joint name='gps0_joint' type='fixed'>
-        <child>gps0::link</child>
+      <joint name='gps_joint' type='fixed'>
+        <child>gps::link</child>
         <parent>base_link</parent>
       </joint>

Commit message: Gps fixed

File: swarm_clover_description/urdf/clover/clover4.xacro (robot description, xacro)
@@ -38,6 +38,6 @@
         <name>gps0</name>
       </include>
-      <joint name='gps_joint' type='fixed'>
-        <child>gps::link</child>
+      <joint name='gps0_joint' type='fixed'>
+        <child>gps0::link</child>
         <parent>base_link</parent>
       </joint>
